File: hardware/Nixie.kicad_sch (KiCad schematic)
At the start: 2 parts

Commit message: Lock in TE CRGH1206F18K as the nixie 18k resistor
Parts:
- R10: footprint (none) -> nixie-esp32:RESC3116X65N; symbol Device:R -> nixie-esp32:CRGH1206F18K; Manufacturer (none) -> TE Connectivity; Manufacturer_Part_Number (none) -> CRGH1206F18K; Power (none) -> 0.5 W; Resistance (none) -> 18 kOhm; Tolerance (none) -> 1%; Voltage_Rating (none) -> 200 V
Connections:
- net +170V: now also R10.2; no longer R10.1
- net at N1.A: now also R10.1; no longer R10.2
Changed lines of the file:
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@@
+	(wire
+		(pts
+			(xy 170.18 67.31) (xy 170.18 80.01)
+		)
+		(stroke
+			(width 0)
+			(type default)
+		)
+	)
 	(wire
 		(pts
@@
 	(wire
 		(pts
-			(xy 170.18 57.15) (xy 170.18 80.01)
-		)
-		(stroke
-			(width 0)
-			(type default)
-		)
-	)
-	(wire
-		(pts
 			(xy 132.08 87.63) (xy 135.89 87.63)
 		)
@@
 	)
 	(symbol
-		(lib_id "Device:R")
-		(at 170.18 53.34 0)
+		(lib_id "nixie-esp32:CRGH1206F18K")
+		(at 170.18 67.31 90)
 		(unit 1)
 		(body_style 1)
@@
 		(fields_autoplaced yes)
 		(property "Reference" "R10"
-			(at 172.72 52.0699 0)
-			(show_name no)
-			(do_not_autoplace no)
-			(effects
-				(font
-					(size 1.27 1.27)
-				)
-				(justify left)
+			(at 172.72 57.1499 90)
+			(show_name no)
+			(do_not_autoplace no)
+			(effects
+				(font
+					(size 1.27 1.27)
+				)
+				(justify right)
 			)
 		)
 		(property "Value" "18k"
-			(at 172.72 54.6099 0)
-			(show_name no)
-			(do_not_autoplace no)
-			(effects
-				(font
-					(size 1.27 1.27)
-				)
-				(justify left)
-			)
-		)
-		(property "Footprint" ""
-			(at 168.402 53.34 90)
+			(at 172.72 59.6899 90)
+			(show_name no)
+			(do_not_autoplace no)
+			(effects
+				(font
+					(size 1.27 1.27)
+				)
+				(justify right)
+			)
+		)
+		(property "Footprint" "nixie-esp32:RESC3116X65N"
+			(at 175.26 58.42 0)
 			(hide yes)
 			(show_name no)
@@
 		)
 		(property "Datasheet" ""
-			(at 170.18 53.34 0)
-			(hide yes)
-			(show_name no)
-			(do_not_autoplace no)
-			(effects
-				(font
-					(size 1.27 1.27)
-				)
-			)
-		)
-		(property "Description" "Resistor"
-			(at 170.18 53.34 0)
-			(hide yes)
-			(show_name no)
+			(at 177.8 58.42 0)
+			(hide yes)
+			(show_name no)
+			(do_not_autoplace no)
+			(effects
+				(font
+					(size 1.27 1.27)
+				)
+			)
+		)
+		(property "Description" "TE Connectivity CRGH1206F18K, 18 kOhm 1% 0.5 W 200 V thick-film resistor, 1206"
+			(at 180.34 58.42 0)
+			(hide yes)
+			(show_name no)
+			(do_not_autoplace no)
+			(effects
+				(font
+					(size 1.27 1.27)
+				)
+			)
+		)
+		(property "Resistance" "18 kOhm"
+			(at 182.88 58.42 0)
+			(hide yes)
+			(show_name no)
+			(do_not_autoplace no)
+			(effects
+				(font
+					(size 1.27 1.27)
+				)
+			)
+		)
+		(property "Tolerance" "1%"
+			(at 185.42 58.42 0)
+			(hide yes)
+			(show_name no)
+			(do_not_autoplace no)
+			(effects
+				(font
+					(size 1.27 1.27)
+				)
+			)
+		)
+		(property "Power" "0.5 W"
+			(at 187.96 58.42 0)
+			(hide yes)
+			(show_name no)
+			(do_not_autoplace no)
+			(effects
+				(font
+					(size 1.27 1.27)
+				)
+			)
+		)
+		(property "Voltage_Rating" "200 V"
+			(at 190.5 58.42 0)
+			(hide yes)
+			(show_name no)
+			(do_not_autoplace no)
+			(effects
+				(font
+					(size 1.27 1.27)
+				)
+			)
+		)
+		(property "Manufacturer" "TE Connectivity"
+			(at 193.04 58.42 0)
+			(hide yes)
+			(show_name no)
+			(do_not_autoplace no)
+			(effects
+				(font
+					(size 1.27 1.27)
+				)
+			)
+		)
+		(property "Manufacturer_Part_Number" "CRGH1206F18K"
+			(at 195.58 58.42 0)
+			(hide yes)
+			(show_name no)

Commit message: Address schematic audit findings
- Move C15 to the ESP32 EN node for proper power-on RC delay and button reset
- Add 10k boot-glitch pull-downs (R13-R16) on the CD4504 level shifter inputs
- Add NCH8200HV input capacitor (C16)
- Switch D2-D4 to the Bivar SMTLA5050RGB symbol/footprint
- Label nixie anode nets and add HV net class with custom DRC clearance rules
- Normalize value formats and assign missing footprints
Connections:
- net ANODE: now reaches N1.A, R10.1
Changed lines of the file:
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@@
 	(generator_version "10.0")
 	(paper "A4")
+	(junction
+		(at 170.18 80.01)
+		(diameter 0)
+		(color 0 0 0 0)
+	)
 	(wire
 		(pts
@@
 	(wire
 		(pts
+			(xy 170.18 80.01) (xy 173.99 80.01)
+		)
+		(stroke
+			(width 0)
+			(type default)
+		)
+	)
+	(wire
+		(pts
 			(xy 132.08 87.63) (xy 135.89 87.63)
 		)
@@
 		)
 	)
+	(label "ANODE"
+		(at 173.99 80.01 0)
+		(effects
+			(font
+				(size 1.27 1.27)
+			)
+			(justify left bottom)
+		)
+	)
