File: hardware/leds.kicad_sch (KiCad schematic)
At the start: 4 parts, among them U3 SN74AHCT1G125DBVR

Commit message: Progress point
Parts:
- C4: renamed from C7; footprint (none) -> Capacitor_SMD:C_0805_2012Metric
- C5: renamed from C8; footprint (none) -> Capacitor_SMD:C_1206_3216Metric
- R7: renamed from R10; footprint (none) -> Resistor_SMD:R_0805_2012Metric
- U3: footprint DBV5 -> nixie-esp32:DBV5
Changed lines of the file:
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@@
 		(dnp no)
 		(fields_autoplaced yes)
-		(property "Reference" "#PWR037"
+		(property "Reference" "#PWR025"
 			(at 208.28 38.1 0)
 			(hide yes)
@@
 			(project "nixie-esp32"
 				(path "/54b4b31b-75dd-48a2-8c91-a3f3099728fc/863e175d-8d38-4d3f-8dde-6bece7eb527a"
-					(reference "#PWR037")
+					(reference "#PWR025")
 					(unit 1)
 				)
@@
 		(dnp no)
 		(fields_autoplaced yes)
-		(property "Reference" "C8"
+		(property "Reference" "C5"
 			(at 212.09 40.6399 0)
 			(show_name no)
@@
 			)
 		)
-		(property "Footprint" ""
+		(property "Footprint" "Capacitor_SMD:C_1206_3216Metric"
 			(at 209.2452 45.72 0)
 			(hide yes)
@@
 			(project "nixie-esp32"
 				(path "/54b4b31b-75dd-48a2-8c91-a3f3099728fc/863e175d-8d38-4d3f-8dde-6bece7eb527a"
-					(reference "C8")
+					(reference "C5")
 					(unit 1)
 				)
@@
 		(dnp no)
 		(fields_autoplaced yes)
-		(property "Reference" "#PWR021"
+		(property "Reference" "#PWR023"
 			(at 179.07 41.91 0)
 			(hide yes)
@@
 			(project "nixie-esp32"
 				(path "/54b4b31b-75dd-48a2-8c91-a3f3099728fc/863e175d-8d38-4d3f-8dde-6bece7eb527a"
-					(reference "#PWR021")
+					(reference "#PWR023")
 					(unit 1)
 				)
@@
 		(dnp no)
 		(fields_autoplaced yes)
-		(property "Reference" "C7"
+		(property "Reference" "C4"
 			(at 101.6 40.6399 0)
 			(show_name no)
@@
 			)
 		)
-		(property "Footprint" ""
+		(property "Footprint" "Capacitor_SMD:C_0805_2012Metric"
 			(at 98.7552 45.72 0)
 			(hide yes)
@@
 			(project "nixie-esp32"
 				(path "/54b4b31b-75dd-48a2-8c91-a3f3099728fc/863e175d-8d38-4d3f-8dde-6bece7eb527a"
-					(reference "C7")
+					(reference "C4")
 					(unit 1)
 				)
@@
 			)
 		)
-		(property "Footprint" "DBV5"
+		(property "Footprint" "nixie-esp32:DBV5"
 			(at 120.65 40.64 0)
 			(hide yes)
@@
 		(dnp no)
 		(fields_autoplaced yes)
-		(property "Reference" "#PWR035"
+		(property "Reference" "#PWR020"
 			(at 97.79 38.1 0)
 			(hide yes)
@@
 			(project "nixie-esp32"
 				(path "/54b4b31b-75dd-48a2-8c91-a3f3099728fc/863e175d-8d38-4d3f-8dde-6bece7eb527a"
-					(reference "#PWR035")
+					(reference "#PWR020")
 					(unit 1)
 				)
@@
 		(dnp no)
 		(fields_autoplaced yes)
-		(property "Reference" "#PWR038"
+		(property "Reference" "#PWR026"
 			(at 208.28 55.88 0)
 			(hide yes)
@@
 			(project "nixie-esp32"
 				(path "/54b4b31b-75dd-48a2-8c91-a3f3099728fc/863e175d-8d38-4d3f-8dde-6bece7eb527a"
-					(reference "#PWR038")
+					(reference "#PWR026")
 					(unit 1)
 				)
@@
 		(dnp no)
 		(fields_autoplaced yes)
-		(property "Reference" "R10"
+		(property "Reference" "R7"
 			(at 185.42 36.83 90)
 			(show_name no)
@@
 			)
 		)
-		(property "Footprint" ""
+		(property "Footprint" "Resistor_SMD:R_0805_2012Metric"
 			(at 185.42 44.958 90)
 			(hide yes)
@@
 			(project "nixie-esp32"
 				(path "/54b4b31b-75dd-48a2-8c91-a3f3099728fc/863e175d-8d38-4d3f-8dde-6bece7eb527a"
-					(reference "R10")
+					(reference "R7")
 					(unit 1)
 				)
@@
 		(dnp no)
 		(fields_autoplaced yes)
-		(property "Reference" "#PWR022"
+		(property "Reference" "#PWR024"
 			(at 179.07 54.61 0)
 			(hide yes)
@@
 			(project "nixie-esp32"
 				(path "/54b4b31b-75dd-48a2-8c91-a3f3099728fc/863e175d-8d38-4d3f-8dde-6bece7eb527a"
-					(reference "#PWR022")
+					(reference "#PWR024")
 					(unit 1)
 				)
@@
 		(dnp no)
 		(fields_autoplaced yes)
-		(property "Reference" "#PWR036"
+		(property "Reference" "#PWR021"
 			(at 97.79 55.88 0)
 			(hide yes)
@@
 			(project "nixie-esp32"
 				(path "/54b4b31b-75dd-48a2-8c91-a3f3099728fc/863e175d-8d38-4d3f-8dde-6bece7eb527a"
-					(reference "#PWR036")
+					(reference "#PWR021")
 					(unit 1)
 				)
@@
 		(dnp no)
 		(fields_autoplaced yes)
-		(property "Reference" "#PWR020"
+		(property "Reference" "#PWR022"
 			(at 115.57 54.61 0)
 			(hide yes)
@@
 			(project "nixie-esp32"
 				(path "/54b4b31b-75dd-48a2-8c91-a3f3099728fc/863e175d-8d38-4d3f-8dde-6bece7eb527a"
-					(reference "#PWR020")
-					(unit 1)
-				)
+					(reference "#PWR022")
+					(unit 1)
+				)

Commit message: Address schematic audit findings
- Move C15 to the ESP32 EN node for proper power-on RC delay and button reset
- Add 10k boot-glitch pull-downs (R13-R16) on the CD4504 level shifter inputs
- Add NCH8200HV input capacitor (C16)
- Switch D2-D4 to the Bivar SMTLA5050RGB symbol/footprint
- Label nixie anode nets and add HV net class with custom DRC clearance rules
- Normalize value formats and assign missing footprints
Parts:
- R7: value 330Ω -> 330
Changed lines of the file:
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@@
 			)
 		)
-		(property "Value" "330Ω"
+		(property "Value" "330"
 			(at 185.42 39.37 90)
 			(show_name no)
