File: hardware/power-12v.kicad_sch (KiCad schematic)
At the start: 7 parts, among them IC1 MCP1661T-E_OT

Commit message: Lock in Coilcraft MSS5131-472MLC as the 12v inductor
Parts:
- L1: footprint (none) -> nixie-esp32:MSS5131; symbol Device:L -> nixie-esp32:MSS5131-472MLC; DCR (none) -> 0.038 Ohm max; Inductance (none) -> 4.7 uH; Irms (none) -> 1.4 A (20 C rise); Manufacturer (none) -> Coilcraft; Manufacturer_Part_Number (none) -> MSS5131-472MLC; Tolerance (none) -> 20%
Changed lines of the file:
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@@
+	)
+	(junction
+		(at 115.57 92.71)
+		(diameter 0)
+		(color 0 0 0 0)
 	)
 	(junction
@@
 	)
 	(junction
-		(at 115.57 85.09)
-		(diameter 0)
-		(color 0 0 0 0)
-	)
-	(junction
 		(at 157.48 76.2)
 		(diameter 0)
@@
 	(wire
 		(pts
+			(xy 130.81 85.09) (xy 121.92 85.09)
+		)
+		(stroke
+			(width 0)
+			(type default)
+		)
+	)
+	(wire
+		(pts
 			(xy 157.48 76.2) (xy 157.48 85.09)
 		)
@@
 	(wire
 		(pts
-			(xy 115.57 85.09) (xy 130.81 85.09)
-		)
-		(stroke
-			(width 0)
-			(type default)
-		)
-	)
-	(wire
-		(pts
 			(xy 157.48 71.12) (xy 157.48 72.39)
 		)
@@
 	(wire
 		(pts
+			(xy 115.57 87.63) (xy 115.57 92.71)
+		)
+		(stroke
+			(width 0)
+			(type default)
+		)
+	)
+	(wire
+		(pts
 			(xy 115.57 124.46) (xy 115.57 127)
 		)
@@
 	(wire
 		(pts
+			(xy 121.92 92.71) (xy 115.57 92.71)
+		)
+		(stroke
+			(width 0)
+			(type default)
+		)
+	)
+	(wire
+		(pts
 			(xy 115.57 127) (xy 115.57 129.54)
 		)
@@
 	(wire
 		(pts
+			(xy 121.92 85.09) (xy 121.92 92.71)
+		)
+		(stroke
+			(width 0)
+			(type default)
+		)
+	)
+	(wire
+		(pts
 			(xy 157.48 87.63) (xy 157.48 85.09)
 		)
@@
 	(wire
 		(pts
-			(xy 115.57 80.01) (xy 115.57 85.09)
-		)
-		(stroke
-			(width 0)
-			(type default)
-		)
-	)
-	(wire
-		(pts
 			(xy 115.57 102.87) (xy 115.57 111.76)
 		)
@@
 	(wire
 		(pts
-			(xy 115.57 85.09) (xy 115.57 95.25)
-		)
-		(stroke
-			(width 0)
-			(type default)
-		)
-	)
-	(wire
-		(pts
 			(xy 139.7 95.25) (xy 130.81 95.25)
 		)
@@
 		(pts
 			(xy 157.48 72.39) (xy 157.48 76.2)
+		)
+		(stroke
+			(width 0)
+			(type default)
+		)
+	)
+	(wire
+		(pts
+			(xy 115.57 92.71) (xy 115.57 95.25)
 		)
 		(stroke
@@
 	)
 	(symbol
-		(lib_id "Device:L")
-		(at 115.57 76.2 0)
+		(lib_id "nixie-esp32:MSS5131-472MLC")
+		(at 115.57 72.39 270)
 		(unit 1)
 		(body_style 1)
@@
 		(fields_autoplaced yes)
 		(property "Reference" "L1"
-			(at 116.84 74.9299 0)
+			(at 116.84 78.7399 90)
 			(show_name no)
 			(do_not_autoplace no)
@@
 		)
 		(property "Value" "4.7µH"
-			(at 116.84 77.4699 0)
+			(at 116.84 81.2799 90)
 			(show_name no)
 			(do_not_autoplace no)
@@
 			)
 		)
-		(property "Footprint" ""
-			(at 115.57 76.2 0)
-			(hide yes)
-			(show_name no)
-			(do_not_autoplace no)
-			(effects
-				(font
-					(size 1.27 1.27)
-				)
-			)
-		)
-		(property "Datasheet" ""
-			(at 115.57 76.2 0)
-			(hide yes)
-			(show_name no)
-			(do_not_autoplace no)
-			(effects
-				(font
-					(size 1.27 1.27)
-				)
-			)
-		)
-		(property "Description" "Inductor"
-			(at 115.57 76.2 0)
-			(hide yes)
-			(show_name no)
+		(property "Footprint" "nixie-esp32:MSS5131"
+			(at 120.65 80.01 0)
+			(hide yes)
+			(show_name no)
+			(do_not_autoplace no)
+			(effects
+				(font
+					(size 1.27 1.27)
+				)
+			)
+		)
+		(property "Datasheet" "${KIPRJMOD}/../datasheets/mss5131.pdf"
+			(at 123.19 80.01 0)
+			(hide yes)
+			(show_name no)
+			(do_not_autoplace no)
+			(effects
+				(font
+					(size 1.27 1.27)
+				)
+			)
+		)
+		(property "Description" "Coilcraft MSS5131-472MLC shielded power inductor, 4.7 uH, 20%, 1.4 A Irms, 0.038 Ohm DCR"
+			(at 125.73 80.01 0)
+			(hide yes)
+			(show_name no)
+			(do_not_autoplace no)
+			(effects
+				(font
+					(size 1.27 1.27)
+				)
+			)
+		)
+		(property "Inductance" "4.7 uH"
+			(at 128.27 80.01 0)
+			(hide yes)
+			(show_name no)
+			(do_not_autoplace no)
+			(effects
+				(font
+					(size 1.27 1.27)
+				)
+			)
+		)
+		(property "Tolerance" "20%"
+			(at 130.81 80.01 0)
+			(hide yes)
+			(show_name no)
+			(do_not_autoplace no)
+			(effects
+				(font
+					(size 1.27 1.27)
+				)
+			)
+		)
+		(property "DCR" "0.038 Ohm max"
+			(at 133.35 80.01 0)
+			(hide yes)
+			(show_name no)
+			(do_not_autoplace no)
+			(effects
+				(font
+					(size 1.27 1.27)
+				)
+			)
+		)
+		(property "Irms" "1.4 A (20 C rise)"
+			(at 135.89 80.01 0)
+			(hide yes)
+			(show_name no)
+			(do_not_autoplace no)
+			(effects
+				(font
+					(size 1.27 1.27)
+				)
+			)
+		)
+		(property "Manufacturer" "Coilcraft"
+			(at 138.43 80.01 0)
+			(hide yes)
+			(show_name no)
+			(do_not_autoplace no)
+			(effects
+				(font
+					(size 1.27 1.27)
+				)
+			)
+		)
+		(property "Manufacturer_Part_Number" "MSS5131-472MLC"
+			(at 140.97 80.01 0)
+			(hide yes)
+			(show_name no)

Commit message: Address schematic audit findings
- Move C15 to the ESP32 EN node for proper power-on RC delay and button reset
- Add 10k boot-glitch pull-downs (R13-R16) on the CD4504 level shifter inputs
- Add NCH8200HV input capacitor (C16)
- Switch D2-D4 to the Bivar SMTLA5050RGB symbol/footprint
- Label nixie anode nets and add HV net class with custom DRC clearance rules
- Normalize value formats and assign missing footprints
Parts:
- C9: value 10µF/25V -> 10µF; Voltage (none) -> 25V
Changed lines of the file:
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@@
 			)
 		)
-		(property "Value" "10µF/25V"
+		(property "Value" "10µF"
 			(at 127 119.38 90)
 			(show_name no)
@@
 			(hide yes)
 			(show_name no)
+			(do_not_autoplace no)
+			(effects
+				(font
+					(size 1.27 1.27)
+				)
+			)
+		)
+		(property "Voltage" "25V"
+			(at 127 121.92 90)
+			(hide yes)
+			(show_name no)
