File: hardware/nixies.kicad_sch (KiCad schematic)
At the start: 0 parts

Commit message: WIP SN74141 redesign
Other:
- removed sheet Power12v
- sheet HvDriver ports: added none; removed BLANK, CLOCK, DATA, LATCH
