File: hardware/nixie-esp32.kicad_pcb (KiCad board)
At the start: 6 copper layers, 70.5 x 70 mm, 53 parts, among them J1 USB4216-03-A_REVA, SW1 RESET, SW2 BOOT, U1 AP7361C-33E-13, U2 ESP32-S3-WROOM-1, U3 SN74AHCT1G125DBVR, U4 SN74141N, U5 SN74141N, U6 SN74141N

Commit message: Improve PCB manufacturing readiness
Other:
- board text added: "JLCJLCJLCJLC"
Changed lines of the file:
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@@
 			(effects
 				(font
-					(size 0.8 0.8)
+					(size 1 1)
 					(thickness 0.15)
 				)
@@
 			(effects
 				(font
-					(size 0.8 0.8)
+					(size 1 1)
 					(thickness 0.15)
 				)
@@
 			(effects
 				(font
-					(size 0.8 0.8)
+					(size 1 1)
 					(thickness 0.15)
 				)
@@
 			(effects
 				(font
-					(size 0.8 0.8)
+					(size 1 1)
 					(thickness 0.15)
 				)
@@
 			(effects
 				(font
-					(size 0.8 0.8)
+					(size 1 1)
 					(thickness 0.15)
 				)
@@
 			(effects
 				(font
-					(size 0.8 0.8)
+					(size 1 1)
 					(thickness 0.15)
 				)
@@
 			(effects
 				(font
-					(size 0.8 0.8)
+					(size 1 1)
 					(thickness 0.15)
 				)
@@
 			(effects
 				(font
-					(size 0.8 0.8)
+					(size 1 1)
 					(thickness 0.15)
 				)
@@
 			(effects
 				(font
-					(size 0.8 0.8)
+					(size 1 1)
 					(thickness 0.15)
 				)
@@
 			(effects
 				(font
-					(size 0.8 0.8)
+					(size 1 1)
 					(thickness 0.15)
 				)
@@
 			(effects
 				(font
-					(size 0.8 0.8)
+					(size 1 1)
 					(thickness 0.15)
 				)
@@
 			(effects
 				(font
-					(size 0.8 0.8)
+					(size 1 1)
 					(thickness 0.15)
 				)
@@
 			(effects
 				(font
-					(size 0.8 0.8)
+					(size 1 1)
 					(thickness 0.15)
 				)
@@
 			(effects
 				(font
-					(size 0.8 0.8)
+					(size 1 1)
 					(thickness 0.15)
 				)
@@
 			(effects
 				(font
-					(size 0.8 0.8)
+					(size 1 1)
 					(thickness 0.15)
 				)
@@
 			(effects
 				(font
-					(size 0.8 0.8)
+					(size 1 1)
 					(thickness 0.15)
 				)
@@
 			(effects
 				(font
-					(size 0.8 0.8)
+					(size 1 1)
 					(thickness 0.15)
 				)
@@
 			(effects
 				(font
-					(size 0.8 0.8)
+					(size 1 1)
 					(thickness 0.15)
 				)
@@
 			(effects
 				(font
-					(size 0.8 0.8)
+					(size 1 1)
 					(thickness 0.15)
 				)
@@
 		(tags "resistor")
 		(property "Reference" "R15"
-			(at 2.9 0 0)
+			(at 3.4 0 0)
 			(layer "B.SilkS")
 			(effects
 				(font
-					(size 0.8 0.8)
+					(size 1 1)
 					(thickness 0.15)
 				)
@@
 			(effects
 				(font
-					(size 0.8 0.8)
+					(size 1 1)
 					(thickness 0.15)
 				)
@@
 			(effects
 				(font
-					(size 0.8 0.8)
+					(size 1 1)
 					(thickness 0.15)
 				)
@@
 			(effects
 				(font
-					(size 0.8 0.8)
+					(size 1 1)
 					(thickness 0.15)
 				)
@@
 			(effects
 				(font
-					(size 0.8 0.8)
+					(size 1 1)
 					(thickness 0.15)
 				)
@@
 		(tags "resistor")
 		(property "Reference" "R16"
-			(at 2.9 -0.2 0)
+			(at 3.4 -0.2 0)
 			(layer "B.SilkS")
 			(effects
 				(font
-					(size 0.8 0.8)
+					(size 1 1)
 					(thickness 0.15)
 				)
@@
 			(effects
 				(font
-					(size 0.8 0.8)
+					(size 1 1)
 					(thickness 0.15)
 				)
@@
 			(effects
 				(font
-					(size 0.8 0.8)
+					(size 1 1)
 					(thickness 0.15)
 				)
@@
 			(polygon
 				(pts
-					(xy 126.84 103.1) (xy 126.84 85.1) (xy 120.89 85.1) (xy 120.89 103.1)
+					(xy 126.84 103.1) (xy 126.84 85.1) (xy 117.5 85.1) (xy 117.5 103.1)
 				)
 			)
@@
 			(effects
 				(font
-					(size 0.8 0.8)
+					(size 1 1)
 					(thickness 0.15)
 				)
@@
 			(effects
 				(font
-					(size 0.8 0.8)
+					(size 1 1)
 					(thickness 0.15)
 				)
@@
 			(effects
 				(font
-					(size 0.8 0.8)
+					(size 1 1)
 					(thickness 0.15)
 				)
@@
 			(effects
 				(font
-					(size 0.8 0.8)
+					(size 1 1)
 					(thickness 0.15)
 				)
@@
 			(effects
 				(font
-					(size 0.8 0.8)
+					(size 1 1)
 					(thickness 0.15)
 				)
@@
 			(effects
 				(font
-					(size 0.8 0.8)
+					(size 1 1)
 					(thickness 0.15)
 				)
@@
 		(tags "resistor")
 		(property "Reference" "R13"
-			(at 2.9 -0.6 0)
+			(at 3.4 -0.6 0)
 			(layer "B.SilkS")
 			(effects
 				(font
-					(size 0.8 0.8)
+					(size 1 1)
 					(thickness 0.15)
 				)
@@
 			(effects
 				(font
-					(size 0.8 0.8)
+					(size 1 1)
 					(thickness 0.15)
 				)
@@
 		)
 	)
-	(gr_text "Rev A  2026-08-30"
-		(at 150.5 97 0)
+	(gr_text "+5V"
+		(at 157.5 104.1 0)
 		(layer "F.SilkS")
 		(effects
@@
 		)
 	)
-	(gr_text "+5V"
-		(at 157.5 104.1 0)
+	(gr_text "+170V"
+		(at 166.1 121.4 0)
 		(layer "F.SilkS")
 		(effects
@@
 		)
 	)
-	(gr_text "+170V"
-		(at 166.1 121.4 0)
+	(gr_text "GND"
+		(at 168 101.3 0)
 		(layer "F.SilkS")
 		(effects
@@
 		)
 	)
-	(gr_text "GND"
-		(at 168 101.3 0)
+	(gr_text "Rev A  2026-08-30"
+		(at 125 94.1 90)
 		(layer "F.SilkS")
 		(effects
@@
 	)
 	(gr_text "nixie-esp32"
-		(at 150.5 94 0)
+		(at 122.2 94.1 90)
 		(layer "F.SilkS")
 		(effects
@@
 		)
 	)
+	(gr_text "JLCJLCJLCJLC"
+		(at 154 145.3 0)
+		(layer "B.SilkS")
+		(effects
+			(font
+				(size 1 1)
+				(thickness 0.15)
+			)
+			(justify mirror)
+		)
+	)
